File: $Laser_Tag.sch (KiCad schematic (older format))
At the start: 20 parts

Commit message: Finished board layout
Parts:
- gave numbers to parts that had none: 20
Connections:
- wire segments 46 -> 40
Changed lines of the file:
@@
 $EndDescr
 $Comp
-L PIC12LF U?
+L PIC12LF U1
 U 1 1 53D52C66
 P 7200 3600
-F 0 "U?" H 7200 3500 60  0000 C CNN
+F 0 "U1" H 7200 3500 60  0000 C CNN
 F 1 "PIC12LF" H 7200 3700 60  0000 C CNN
 F 2 "" H 7200 3600 60  0000 C CNN
@@
 $EndComp
 $Comp
-L VDD #PWR?
+L VDD #PWR11
 U 1 1 53D52EF1
 P 6150 3100
-F 0 "#PWR?" H 6150 3200 30  0001 C CNN
+F 0 "#PWR11" H 6150 3200 30  0001 C CNN
 F 1 "VDD" H 6150 3210 30  0000 C CNN
 F 2 "" H 6150 3100 60  0000 C CNN
@@
 $EndComp
 $Comp
-L GND #PWR?
+L GND #PWR12
 U 1 1 53D52F03
 P 8550 3350
-F 0 "#PWR?" H 8550 3350 30  0001 C CNN
+F 0 "#PWR12" H 8550 3350 30  0001 C CNN
 F 1 "GND" H 8550 3280 30  0001 C CNN
 F 2 "" H 8550 3350 60  0000 C CNN
@@
 $EndComp
 $Comp
-L SPEAKER SP?
+L SPEAKER SP1
 U 1 1 53D52F16
 P 10000 5500
-F 0 "SP?" H 9900 5750 70  0000 C CNN
+F 0 "SP1" H 9900 5750 70  0000 C CNN
 F 1 "SPEAKER" H 9900 5250 70  0000 C CNN
 F 2 "~" H 10000 5500 60  0000 C CNN
@@
 MIC_IN
 $Comp
-L MICROPHONE M?
+L MICROPHONE M1
 U 1 1 53D52F41
 P 2700 6000
-F 0 "M?" H 2700 5750 60  0000 C CNN
+F 0 "M1" H 2700 5750 60  0000 C CNN
 F 1 "MICROPHONE" H 2700 6250 60  0000 C CNN
 F 2 "" H 2700 6000 60  0000 C CNN
@@
 $EndComp
 $Comp
-L R R?
+L R R1
 U 1 1 53D52F5A
 P 3000 5400
-F 0 "R?" V 3080 5400 40  0000 C CNN
+F 0 "R1" V 3080 5400 40  0000 C CNN
 F 1 "2.2K" V 3007 5401 40  0000 C CNN
 F 2 "~" V 2930 5400 30  0000 C CNN
@@
 $EndComp
 $Comp
-L VDD #PWR?
+L VDD #PWR5
 U 1 1 53D52F73
 P 3850 5000
-F 0 "#PWR?" H 3850 5100 30  0001 C CNN
+F 0 "#PWR5" H 3850 5100 30  0001 C CNN
 F 1 "VDD" H 3850 5110 30  0000 C CNN
 F 2 "" H 3850 5000 60  0000 C CNN
@@
 $EndComp
 $Comp
-L GND #PWR?
+L GND #PWR2
 U 1 1 53D52F95
 P 3000 6200
-F 0 "#PWR?" H 3000 6200 30  0001 C CNN
+F 0 "#PWR2" H 3000 6200 30  0001 C CNN
 F 1 "GND" H 3000 6130 30  0001 C CNN
 F 2 "" H 3000 6200 60  0000 C CNN
@@
 $EndComp
 $Comp
-L C C?
+L C C1
 U 1 1 53D52FAF
 P 3400 5950
-F 0 "C?" H 3400 6050 40  0000 L CNN
+F 0 "C1" H 3400 6050 40  0000 L CNN
 F 1 "1uF" H 3406 5865 40  0000 L CNN
 F 2 "~" H 3438 5800 30  0000 C CNN
@@
 $EndComp
 $Comp
-L NPN Q?
+L NPN Q1
 U 1 1 53D52FCA
 P 3800 5950
-F 0 "Q?" H 3800 5800 50  0000 R CNN
+F 0 "Q1" H 3800 5800 50  0000 R CNN
 F 1 "2N3904" H 3800 6100 50  0000 R CNN
 F 2 "~" H 3800 5950 60  0000 C CNN
@@
 $EndComp
 $Comp
-L R R?
+L R R4
 U 1 1 53D52FD9
 P 4100 5350
-F 0 "R?" V 4180 5350 40  0000 C CNN
+F 0 "R4" V 4180 5350 40  0000 C CNN
 F 1 "10K" V 4107 5351 40  0000 C CNN
 F 2 "~" V 4030 5350 30  0000 C CNN
@@
 $EndComp
 $Comp
-L R R?
+L R R3
 U 1 1 53D52FE8
 P 3850 5600
-F 0 "R?" V 3930 5600 40  0000 C CNN
+F 0 "R3" V 3930 5600 40  0000 C CNN
 F 1 "100K" V 3857 5601 40  0000 C CNN
 F 2 "~" V 3780 5600 30  0000 C CNN
@@
 $EndComp
 $Comp
-L GND #PWR?
+L GND #PWR6
 U 1 1 53D52FF7
 P 3900 6200
-F 0 "#PWR?" H 3900 6200 30  0001 C CNN
+F 0 "#PWR6" H 3900 6200 30  0001 C CNN
 F 1 "GND" H 3900 6130 30  0001 C CNN
 F 2 "" H 3900 6200 60  0000 C CNN
@@
 $EndComp
 $Comp
-L C C?
+L C C3
 U 1 1 53D53243
 P 4550 5750
-F 0 "C?" H 4550 5850 40  0000 L CNN
+F 0 "C3" H 4550 5850 40  0000 L CNN
 F 1 ".1uF" H 4556 5665 40  0000 L CNN
 F 2 "~" H 4588 5600 30  0000 C CNN
@@
 MIC_IN
 $Comp
-L PHOTODETECTOR P?
+L PHOTODETECTOR P1
 U 1 1 53D5376D
 P 3000 2600
-F 0 "P?" H 3000 2300 60  0000 C CNN
+F 0 "P1" H 3000 2300 60  0000 C CNN
 F 1 "PHOTODETECTOR" H 3000 3000 60  0000 C CNN
 F 2 "" H 3000 2600 60  0000 C CNN
@@
 $EndComp
 $Comp
-L VDD #PWR?
+L VDD #PWR3
 U 1 1 53D5377A
 P 3550 1750
-F 0 "#PWR?" H 3550 1850 30  0001 C CNN
+F 0 "#PWR3" H 3550 1850 30  0001 C CNN
 F 1 "VDD" H 3550 1860 30  0000 C CNN
 F 2 "" H 3550 1750 60  0000 C CNN
@@
 $EndComp
 $Comp
-L C C?
+L C C2
 U 1 1 53D53799
 P 3850 2550
-F 0 "C?" H 3850 2650 40  0000 L CNN
+F 0 "C2" H 3850 2650 40  0000 L CNN
 F 1 "1uF" H 3856 2465 40  0000 L CNN
 F 2 "~" H 3888 2400 30  0000 C CNN
@@
 IR_IN
 $Comp
-L R R?
+L R R2
 U 1 1 53D53896
 P 3550 2000
-F 0 "R?" V 3630 2000 40  0000 C CNN
+F 0 "R2" V 3630 2000 40  0000 C CNN
 F 1 "330" V 3557 2001 40  0000 C CNN
 F 2 "~" V 3480 2000 30  0000 C CNN
@@
 $EndComp
 $Comp
-L LED D?
+L LED D4
 U 1 1 53D53960
 P 8900 3500
-F 0 "D?" H 8900 3600 50  0000 C CNN
+F 0 "D4" H 8900 3600 50  0000 C CNN
 F 1 "IR OUT" H 8900 3400 50  0000 C CNN
 F 2 "~" H 8900 3500 60  0000 C CNN
@@
 	3900 6150 3900 6200
 Wire Wire Line
-	3000 5000 3850 5000
-Wire Wire Line
-	3850 5000 4100 5000
+	3000 5000 4100 5000
 Wire Wire Line
 	4100 5000 4100 5100
@@
 	3600 5600 3600 5950
 Wire Wire Line
-	3900 5750 4100 5750
-Wire Wire Line
-	4100 5750 4350 5750
+	3900 5750 4350 5750
 Wire Wire Line
 	4100 5750 4100 5600
@@
 	4750 5750 5050 5750
 Wire Wire Line
-	3300 2350 3550 2350
-Wire Wire Line
-	3550 2350 3850 2350
+	3300 2350 3850 2350
 Wire Wire Line
 	3550 2350 3550 2250
@@
 SPEAKER
 $Comp
-L VDD #PWR?
+L VDD #PWR14
 U 1 1 53D53BD1
 P 9500 5250
-F 0 "#PWR?" H 9500 5350 30  0001 C CNN
+F 0 "#PWR14" H 9500 5350 30  0001 C CNN
 F 1 "VDD" H 9500 5360 30  0000 C CNN
 F 2 "" H 9500 5250 60  0000 C CNN
@@
 	9500 5400 9700 5400
 $Comp
-L LED D?
+L LED D2
 U 1 1 53D53DD8
 P 5400 3500
-F 0 "D?" H 5400 3600 50  0000 C CNN
+F 0 "D2" H 5400 3600 50  0000 C CNN
 F 1 "LED" H 5400 3400 50  0000 C CNN
 F 2 "~" H 5400 3500 60  0000 C CNN
@@
 $EndComp
 $Comp
-L LED D?
+L LED D3
 U 1 1 53D53DF9
 P 5400 3900
-F 0 "D?" H 5400 4000 50  0000 C CNN
+F 0 "D3" H 5400 4000 50  0000 C CNN
 F 1 "LED" H 5400 3800 50  0000 C CNN
 F 2 "~" H 5400 3900 60  0000 C CNN
@@
 $EndComp
 $Comp
-L VDD #PWR?
+L VDD #PWR8
 U 1 1 53D53E42
 P 5200 3500
-F 0 "#PWR?" H 5200 3600 30  0001 C CNN
+F 0 "#PWR8" H 5200 3600 30  0001 C CNN
 F 1 "VDD" H 5200 3610 30  0000 C CNN
 F 2 "" H 5200 3500 60  0000 C CNN
@@
 $EndComp
 $Comp
-L VDD #PWR?
+L VDD #PWR9
 U 1 1 53D53E51
 P 5200 3900
-F 0 "#PWR?" H 5200 4000 30  0001 C CNN
+F 0 "#PWR9" H 5200 4000 30  0001 C CNN
 F 1 "VDD" H 5200 4010 30  0000 C CNN
 F 2 "" H 5200 3900 60  0000 C CNN
@@
 	5600 3900 6150 3900
 $Comp
-L BATTERY BT?
+L BATTERY BT1
 U 1 1 53D54000
 P 3350 3800
-F 0 "BT?" H 3350 4000 50  0000 C CNN
+F 0 "BT1" H 3350 4000 50  0000 C CNN
 F 1 "BATTERY" H 3350 3610 50  0000 C CNN
 F 2 "~" H 3350 3800 60  0000 C CNN
@@
 $EndComp
 $Comp
-L GND #PWR?
+L GND #PWR4
 U 1 1 53D5401E
 P 3750 3950
-F 0 "#PWR?" H 3750 3950 30  0001 C CNN
+F 0 "#PWR4" H 3750 3950 30  0001 C CNN
 F 1 "GND" H 3750 3880 30  0001 C CNN
 F 2 "" H 3750 3950 60  0000 C CNN
@@
 	3750 3800 3750 3950
 $Comp
-L VDD #PWR?
+L VDD #PWR1
 U 1 1 53D5404F
 P 2950 3650
-F 0 "#PWR?" H 2950 3750 30  0001 C CNN
+F 0 "#PWR1" H 2950 3750 30  0001 C CNN
 F 1 "VDD" H 2950 3760 30  0000 C CNN
 F 2 "" H 2950 3650 60  0000 C CNN
@@
 	2950 3800 2950 3650
 $Comp
-L SW_PUSH SW?
+L SW_PUSH SW1
 U 1 1 53D548CF
 P 5400 4650
-F 0 "SW?" H 5550 4760 50  0000 C CNN
+F 0 "SW1" H 5550 4760 50  0000 C CNN
 F 1 "SW_PUSH" H 5400 4570 50  0000 C CNN
 F 2 "~" H 5400 4650 60  0000 C CNN
@@
 MIC_IN
 $Comp
-L VDD #PWR?
+L VDD #PWR7
 U 1 1 53D5492C
 P 4600 4500
-F 0 "#PWR?" H 4600 4600 30  0001 C CNN
+F 0 "#PWR7" H 4600 4600 30  0001 C CNN
 F 1 "VDD" H 4600 4610 30  0000 C CNN
 F 2 "" H 4600 4500 60  0000 C CNN
@@
 	4600 4650 4600 4500
 $Comp
-L DIODE D?
+L DIODE D1
 U 1 1 53D54A1B
 P 5250 5750
-F 0 "D?" H 5250 5850 40  0000 C CNN
+F 0 "D1" H 5250 5850 40  0000 C CNN
 F 1 "DIODE" H 5250 5650 40  0000 C CNN
 F 2 "~" H 5250 5750 60  0000 C CNN
@@
 $EndComp
 $Comp
-L C C?
+L C C4
 U 1 1 53D54A2A
 P 5650 5950
-F 0 "C?" H 5650 6050 40  0000 L CNN
+F 0 "C4" H 5650 6050 40  0000 L CNN
 F 1 ".33uF" H 5656 5865 40  0000 L CNN
 F 2 "~" H 5688 5800 30  0000 C CNN
@@
 $EndComp
 $Comp
-L R R?
+L R R5
 U 1 1 53D54A39
 P 5950 6000
-F 0 "R?" V 6030 6000 40  0000 C CNN
+F 0 "R5" V 6030 6000 40  0000 C CNN
 F 1 "10K" V 5957 6001 40  0000 C CNN
 F 2 "~" V 5880 6000 30  0000 C CNN
@@
 $EndComp
 Wire Wire Line
-	5450 5750 5650 5750
-Wire Wire Line
-	5650 5750 5950 5750
-Wire Wire Line
-	5950 5750 6350 5750
+	5450 5750 6350 5750
 Connection ~ 5650 5750
 Wire Wire Line
 	5650 6150 5650 6250
 Wire Wire Line
-	5650 6250 5800 6250
-Wire Wire Line
-	5800 6250 5950 6250
-$Comp
-L GND #PWR?
+	5650 6250 5950 6250
+$Comp
+L GND #PWR10
 U 1 1 53D54AC4
 P 5800 6350
-F 0 "#PWR?" H 5800 6350 30  0001 C CNN
+F 0 "#PWR10" H 5800 6350 30  0001 C CNN
 F 1 "GND" H 5800 6280 30  0001 C CNN
 F 2 "" H 5800 6350 60  0000 C CNN
@@
 	9100 3500 9350 3500
 $Comp
-L GND #PWR?
+L GND #PWR13
 U 1 1 53D53A84
 P 9350 3550
-F 0 "#PWR?" H 9350 3550 30  0001 C CNN
+F 0 "#PWR13" H 9350 3550 30  0001 C CNN
 F 1 "GND" H 9350 3480 30  0001 C CNN
 F 2 "" H 9350 3550 60  0000 C CNN
